Commit message: tesrbringup

File: robot_ws/src/robot_bringup/urdf/robot.urdf.xacro (robot description, xacro)
@@ -1,18 +1,42 @@
-<?xml version="1.0"?>
-<robot name="kbot">
-    <!-- link -->
-    <link name="base_footprint"/>
-    <link name="base_link"/>
-    <link name="base_scan"/>
-    <!-- joint -->
-    <joint name="base_joint" type="fixed">
-        <parent link="base_footprint"/>
-        <child link="base_link"/>
-        <origin xyz="0.0 0.0 0.090" rpy="0.0 0.0 0.0"/>
-    </joint>
-    <joint name="scan_joint" type="fixed">
-        <parent link="base_link"/>
-        <child link="base_scan"/>
-        <origin xyz="-0.095 0.0 0.073" rpy="0.0 0.0 3.1415925359"/>
-    </joint>
+<?xml version="1.0" encoding="utf-8" ?>
+<robot name="ironx" xmlns:xacro="http://ros.org/wiki/xacro">
+	<xacro:include filename="$(find tesr_ros_ironx_driver_pkg)/urdf/tesr_ironx.gazebo.urdf"/>
+	<link name="base_footprint"/>
+	<link name="base_link">
+		<visual>
+			<origin xyz="0.12645 0.125 0" rpy="1.5708 0 -1.5708"/>
+			<geometry> <mesh filename="package://tesr_ros_ironx_driver_pkg/meshes/tesr_ros_ironx.STL" scale="0.001 0.001 0.001"/>
+			</geometry>
+			<material name=""> <color rgba="1 1 1 1" />
+			</material>
+		</visual>
+		<collision>
+			<origin xyz="0.12645 0.125 0" rpy="1.5708 0 -1.5708"/>
+			<geometry> <mesh filename="package://tesr_ros_ironx_driver_pkg/meshes/tesr_ros_ironx.STL" scale="0.001 0.001 0.001"/>
+			</geometry>
+		</collision>
+		<inertial>
+			<origin xyz="0 0 0"/>
+			<mass value="0.05"/>
+			<inertia ixx="2.2124416e-03" ixy="-1.2294101e-05" ixz="3.4938785e-05"
+				iyy="2.1193702e-03" iyz="-5.0120904e-06" izz="2.0064271e-03"/>
+		</inertial>
+	</link>
+	<joint name="base_joint" type="fixed">
+		<parent link="base_footprint"/>
+		<child link="base_link"/>
+		<origin xyz="0.0 0.0 0.0" rpy="0 0 0"/>
+	</joint>
+	<link name="imu_link"/>
+	<link name="base_scan"/>
+	<joint name="imu_joint" type="fixed">
+		<parent link="base_link"/>
+		<child link="imu_link"/>
+		<origin xyz="-0.02 0.03 0.08212" rpy="0 0 0"/>
+	</joint>
+	<joint name="scan_joint" type="fixed">
+		<parent link="base_link"/>
+		<child link="base_scan"/>
+		<origin xyz="0 0.1 0.168" rpy="0 0 0"/>
+	</joint>
 </robot>

Commit message: update movetogoal

File: robot_ws/src/robot_bringup/urdf/robot.urdf.xacro (robot description, xacro)
@@ -1,26 +1,8 @@
 <?xml version="1.0" encoding="utf-8" ?>
 <robot name="ironx" xmlns:xacro="http://ros.org/wiki/xacro">
-	<xacro:include filename="$(find tesr_ros_ironx_driver_pkg)/urdf/tesr_ironx.gazebo.urdf"/>
 	<link name="base_footprint"/>
-	<link name="base_link">
-		<visual>
-			<origin xyz="0.12645 0.125 0" rpy="1.5708 0 -1.5708"/>
-			<geometry> <mesh filename="package://tesr_ros_ironx_driver_pkg/meshes/tesr_ros_ironx.STL" scale="0.001 0.001 0.001"/>
-			</geometry>
-			<material name=""> <color rgba="1 1 1 1" />
-			</material>
-		</visual>
-		<collision>
-			<origin xyz="0.12645 0.125 0" rpy="1.5708 0 -1.5708"/>
-			<geometry> <mesh filename="package://tesr_ros_ironx_driver_pkg/meshes/tesr_ros_ironx.STL" scale="0.001 0.001 0.001"/>
-			</geometry>
-		</collision>
-		<inertial>
-			<origin xyz="0 0 0"/>
-			<mass value="0.05"/>
-			<inertia ixx="2.2124416e-03" ixy="-1.2294101e-05" ixz="3.4938785e-05"
-				iyy="2.1193702e-03" iyz="-5.0120904e-06" izz="2.0064271e-03"/>
-		</inertial>
-	</link>
+	<link name="base_link"/>
+	<link name="imu_link"/>
+	<link name="base_scan"/>
 	<joint name="base_joint" type="fixed">
 		<parent link="base_footprint"/>
@@ -28,6 +10,4 @@
 		<origin xyz="0.0 0.0 0.0" rpy="0 0 0"/>
 	</joint>
-	<link name="imu_link"/>
-	<link name="base_scan"/>
 	<joint name="imu_joint" type="fixed">
 		<parent link="base_link"/>
@@ -38,5 +18,5 @@
 		<parent link="base_link"/>
 		<child link="base_scan"/>
-		<origin xyz="0 0.1 0.168" rpy="0 0 0"/>
+		<origin xyz="0 0.1 0.168" rpy="0 0 3.141592653"/>
 	</joint>
 </robot>
